Commit message: Change scythe color Alter talos right arm robot

File: pyphysx_envs/robot_data/talos_desription/talos_body_right_arm.urdf (robot description, URDF)
Before this commit: robot talos, 11 links, 10 joints
Links:
- added link tool_link
Joints:
- added joint talos_spade_joint: type revolute, parent wrist_right_ft_link, child tool_link, origin xyz=0 0 -0.05 rpy=1.57079632679 0 -3.14, axis 0 0 1, limit lower=-6.14 upper=6.14 effort=30 velocity=1.0
