Commit message: Update from cluster changes

File: pyphysx_envs/robot_data/panda_description/panda_no_hand.urdf (robot description, URDF)
Before this commit: robot panda, 8 links, 7 joints
Links:
- added link panda_holder; collision cylinder length=0.003 radius=0.04; visual cylinder length=0.03 radius=0.04
Joints:
- added joint panda_spade_joint: type fixed, parent panda_link7, child panda_holder, origin xyz=0 0 0.1 rpy=0 0 0

File: pyphysx_envs/robot_data/talos_desription/talos_body_right_arm.urdf (robot description, URDF)
Before this commit: robot talos, 12 links, 11 joints
Links:
- added link panda_holder; collision cylinder length=0.0003 radius=0.04; visual cylinder length=0.03 radius=0.04
Joints:
- added joint panda_spade_joint: type fixed, parent tool_link, child panda_holder, origin xyz=0.0 0.01 0. rpy=1.57079632679 0 0

File: pyphysx_envs/robot_data/ur_description/ur5_robot_no_tool.urdf (robot description, URDF)
Before this commit: robot ur5, 8 links, 7 joints
Links:
- added link panda_holder; collision cylinder length=0.003 radius=0.04; visual cylinder length=0.03 radius=0.04
Joints:
- added joint panda_spade_joint: type fixed, parent ee_link, child panda_holder, origin xyz=0.01 0. 0 rpy=0 1.57079632679 0
